Commit message: test(safety): replace ignored robot-v1 test with fixture-driven coverage
The framework-level range-classification logic (downward ToF →
Cliff, forward ToF → Obstacle) had been demonstrated via a test
reaching into `models/robot-v1/`. After the repo split that path
is gone and the test was #[ignore]d.

Rebuild it on top of `fixture/robot/<bundle>` so the framework
exercises its own classification logic without touching any
specific robot.

Signed-off-by: jbernavaprah <webjure@gmail.com>

File: fixture/robot/lowrate-range-diff-drive/structure.urdf (robot description, URDF)
Before this commit: robot RgbdImuDiffDrive, 9 links, 8 joints
Links:
- added link ground_tof_mount
Joints:
- added joint ground_tof_mount_joint: type fixed, parent base_link, child ground_tof_mount, origin xyz=0.12 0 0.03 rpy=0 1.5708 0
